Commit message: fix with working in moveit

File: Robot_ros2_ws/src/aar6/urdf/PAROL6.urdf (robot description, URDF)
Before this commit: robot aar6, 11 links, 10 joints
Joints:
- joint ee_link: type revolute -> fixed

Commit message: fix with wodden board and cv stuff

File: Robot_ros2_ws/src/aar6/urdf/PAROL6.urdf (robot description, URDF)
Before this commit: robot aar6, 11 links, 10 joints
Links:
- added link wooden_base, mass 5.0; collision mesh filename=package://aar6/meshes/wodeen_base.dae; visual mesh filename=package://aar6/meshes/wodeen_base.dae
Joints:
- added joint world_to_wooden_base: type fixed, parent world, child wooden_base, origin xyz=0.0 0.0 0.0 rpy=0 0 0
- joint L1: limit lower=-1.7 upper=1.7 effort=300 velocity=3 -> lower=-3.142 upper=3.142 effort=300 velocity=15
- joint L2: limit lower=-0.98 upper=1 effort=300 velocity=3 -> lower=-0.98 upper=1 effort=300 velocity=15
- joint L3: limit lower=-2 upper=1.3 effort=300 velocity=3 -> lower=-2 upper=1.3 effort=300 velocity=15
- joint L4: limit lower=-2 upper=2 effort=300 velocity=3 -> lower=-4.9 upper=0.3 effort=300 velocity=15
- joint L5: limit lower=-2.1 upper=2.1 effort=300 velocity=3 -> lower=-2.1 upper=2.1 effort=300 velocity=15
- joint L6: limit lower=-3.1 upper=3.1 effort=300 velocity=3 -> lower=-3.1 upper=3.1 effort=300 velocity=15
- joint base_joint: origin xyz=0.0 0.0 0.00 rpy=0 0 0 -> xyz=0.145 0.0 0.069 rpy=0 0 3.142; parent world -> wooden_base
